File: hardware/IO_board/IO.brd (EAGLE design)
At the start: 167.9 x 122.5 mm, 52 parts, among them IC1 MAX232, IC4 74HCT139N, IC5 74AC06N, IC7 MAX232, J1 DIN5, X2 CRYSTALS-NOGND-CFPX-217

Commit message: CPU board and I/O board update
Parts:
- added IC10, IC8, IC9: 74HCT245DW, 74xx-eu:SO20W
- R7: device rcl:0204/5 -> rcl:0204/7
- moved BATTERY_1 168.8 mm to (4.76, 37.8), turned to 270 degrees
- moved D1 167.4 mm to (7.30, 60.0)
- moved D2 154.1 mm to (22.2, 59.4), turned to 90 degrees
- moved C23 135.2 mm to (26.4, 60.3), turned to 180 degrees
- moved C3 133.7 mm to (17.8, 64.5)
- moved C20 131.6 mm to (26.4, 57.8), turned to 180 degrees
- moved U$2 130.4 mm to (36.2, 65.4), turned to 90 degrees
- moved X2 128.9 mm to (29.5, 59.1), turned to 90 degrees
- moved R10 111.6 mm to (37.8, 55.9), turned to 270 degrees
- moved IC2 44.4 mm to (66.7, 56.5)
- moved C2 42.5 mm to (63.2, 60.3)
- moved C1 22.5 mm to (128.1, 69.2), turned to 0 degrees
- moved R7 21.6 mm to (114.9, 110.8)
- moved IC5 20.5 mm to (108.0, 104.8)
- moved R9 20.5 mm to (109.5, 110.7)
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Connections:
- new net !IORQ_IN: IC9.8, SV2.44
- new net A0_IN: IC10.2, SV2.15
- new net A1_IN: IC10.3, SV2.16
- new net A2_IN: IC10.4, SV2.17
- new net A3_IN: IC10.5, SV2.18
- new net A4_IN: IC10.6, SV2.19
- new net CLK_IN: IC9.4, SV2.36
- new net D0_IN: IC8.2, SV2.7
- new net D1_IN: IC8.3, SV2.8
- new net D2_IN: IC8.4, SV2.9
- new net D3_IN: IC8.5, SV2.10
- new net D4_IN: IC8.6, SV2.11
- new net D5_IN: IC8.7, SV2.12
- new net D6_IN: IC8.8, SV2.13
- new net D7_IN: IC8.9, SV2.14
- new net M1_IN: IC9.9, SV2.43
- new net RD_IN: IC9.2, SV2.34
- new net WR_IN: IC9.3, SV2.35
- net !IORQ: now also IC9.12; no longer SV2.44
- net A0: now also IC10.18; no longer SV2.15
- net A1: now also IC10.17; no longer SV2.16
- net A2: now also IC10.16; no longer SV2.17
- net A3: now also IC10.15; no longer SV2.18
- net A4: now also IC10.14; no longer SV2.19
- net CLK: now also IC9.16; no longer SV2.36
- net D0: now also IC8.18; no longer SV2.7
- net D1: now also IC8.17; no longer SV2.8
- net D2: now also IC8.16; no longer SV2.9
- net D3: now also IC8.15; no longer SV2.10
- net D4: now also IC8.14; no longer SV2.11
- net D5: now also IC8.13; no longer SV2.12
- net D6: now also IC8.12; no longer SV2.13
- net D7: now also IC8.11; no longer SV2.14
- net GND: now also IC10.10, IC10.19, IC10.7, IC10.8, IC10.9, IC8.10, IC8.19, IC9.10, IC9.19, IC9.5, IC9.6, IC9.7
- net M1: now also IC9.11; no longer SV2.43
- net RD: now also IC8.1, IC9.18; no longer SV2.34
- net VCC: now also IC10.20, IC8.20, IC9.20
- net WR: now also IC9.17; no longer SV2.35
Routing:
- net !IORQ: track 176.4 -> 83.9 mm
- net A1: track 189.5 -> 100.9 mm, vias 3 -> 2
- net A0: track 199.2 -> 123.0 mm, vias 4 -> 2
- net D7: track 151.9 -> 77.7 mm
- net D5: track 149.8 -> 75.6 mm
- net D4: track 129.9 -> 58.8 mm
- net D6: track 132.0 -> 60.9 mm
- net CLK: track 174.5 -> 104.0 mm
- net M1: track 166.3 -> 95.9 mm, vias 0 -> 2
- net D3: track 174.3 -> 112.3 mm, vias 3 -> 2
- net INT: track 182.4 -> 124.6 mm, vias 2 -> 4
- net D1: track 194.0 -> 136.4 mm, vias 3 -> 2
- net !RESET: track 218.6 -> 161.8 mm
- net UART_CS: track 72.3 -> 20.8 mm, vias 3 -> 1
- net RTC_IRQ: track 50.7 -> 0.00 mm
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
Commit message: I/O board updated (work in progress)
Parts:
- added C30, C31, C32: 100N, rcl:C0603
- added IC11: 74HCT393N, 74xx-eu:DIL14
- added QG1: (no value), crystal:DIL14S
- added R1: (no value), rcl:R0603
- moved C21 170.3 mm to (8.26, 96.6), turned to 270 degrees
- moved C24 159.3 mm to (48.9, 84.8)
- moved C17 154.7 mm to (128.1, 54.0), turned to 0 degrees
- moved C18 135.5 mm to (22.0, 55.2), turned to 0 degrees
- moved C13 118.9 mm to (32.4, 52.8), turned to 90 degrees
- moved C19 103.5 mm to (116.3, 65.4), turned to 0 degrees
- moved BATTERY_1 28.7 mm to (18.7, 62.9), turned to 0 degrees
- moved D1 18.4 mm to (25.7, 59.1), turned to 90 degrees
- moved C3 17.5 mm to (35.1, 62.0), turned to 270 degrees
- moved IC4 12.7 mm to (136.5, 22.2)
- moved C16 11.7 mm to (137.2, 31.1)
- moved D2 6.04 mm to (28.3, 59.1)
- moved R19 1.27 mm to (94.9, 104.8)
- moved C7 0.63 mm to (128.9, 107.0)
- moved C8 0.63 mm to (124.7, 110.1)
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Connections:
- new net BAUDRATE: IC11.10, IC2.13, IC2.14, IC2.27
- new net N$26: IC11.1, QG1.8
- new net N$27: IC11.13, IC11.6
- new net N$30: QG1.1, R1.2
- new net N$32: IC2.7, IC6.13
- net A4: no longer IC4.2
- net CS_1: no longer IC4.1
- net GND: now also C30.2, C31.2, C32.2, IC11.12, IC11.2, IC11.7, IC4.1, IC4.2, IC5.5, QG1.7
- net TIMER_CS: now also IC6.16
- net UART_CS: now also IC2.35
- net VCC: now also C30.1, C31.1, C32.1, IC10.1, IC11.14, IC9.1, QG1.14, R1.1
Routing:
- net VCC: track 422.2 -> 645.3 mm, vias 6 -> 14
- net CS_0: track 0.00 -> 176.3 mm, vias 0 -> 2
- net A2: track 0.00 -> 171.5 mm, vias 0 -> 4
- net A3: track 15.1 -> 186.0 mm, vias 1 -> 4
- net UART_CS: track 20.8 -> 111.5 mm, vias 1 -> 2
- net A1: track 100.9 -> 174.9 mm, vias 2 -> 4
- net N$32: track 0.00 -> 67.2 mm, vias 0 -> 2
- net BAUDRATE: track 0.00 -> 48.7 mm
- net A4: track 23.9 -> 65.9 mm, vias 1 -> 2
- net KBD_CS: track 106.8 -> 139.0 mm, vias 3 -> 2
- net CS_DMA: track 27.3 -> 0.00 mm, vias 1 -> 0
- net CS_INT: track 25.7 -> 0.00 mm, vias 1 -> 0
- net TIMER_CS: track 22.1 -> 46.9 mm, vias 1 -> 2
- net N$26: track 0.00 -> 18.5 mm
- net CS_1: track 16.8 -> 0.00 mm
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
Commit message: IO board update (work in progress)
Parts:
- added R2: (no value), rcl:R0603
- added R3: (no value), rcl:0207/15
Connections:
- new net N$34: IC2.16, IC2.19, IC2.22, IC2.25, R3.1
- new net N$36: IC2.10, IC2.11, IC2.29, IC2.30, R2.1
- net VCC: now also R2.2, R3.2
Routing:
- net GND: track 91.5 -> 138.2 mm, vias 18 -> 20
- net N$34: track 0.00 -> 40.8 mm, vias 0 -> 2
- net N$36: track 0.00 -> 22.9 mm
- net VCC: track 645.3 -> 643.0 mm
- net BAUDRATE: track 48.7 -> 48.2 mm, vias 0 -> 2
Changed lines of the file:
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@@
 <element name="C32" library="rcl" package="C0603" value="100N" x="40.005" y="50.165" rot="MR90"/>
 <element name="R1" library="rcl" package="R0603" value="" x="23.495" y="47.625" rot="MR0"/>
+<element name="R2" library="rcl" package="R0603" value="" x="56.515" y="58.6486" rot="MR90"/>
+<element name="R3" library="rcl" package="0207/15" value="" x="54.61" y="50.165" rot="R90"/>
 </elements>
 <signals>
@@
 <contactref element="C31" pad="2"/>
 <contactref element="C32" pad="2"/>
+<via x="94.615" y="58.166" extent="1-16" drill="0.6" diameter="1.4224" shape="octagon"/>
+<wire x1="94.615" y1="58.166" x2="94.615" y2="11.4935" width="0.6096" layer="1"/>
+<via x="94.615" y="11.4935" extent="1-16" drill="0.6" diameter="1.4224" shape="octagon"/>
 </signal>
 <signal name="N$37">
@@
 <wire x1="52.07" y1="86.36" x2="52.07" y2="60.325" width="0.6096" layer="1"/>
 <via x="52.07" y="60.325" extent="1-16" drill="0.6" diameter="1.778" shape="octagon"/>
-<wire x1="59.055" y1="60.325" x2="52.07" y2="60.325" width="1.016" layer="16"/>
-<wire x1="52.07" y1="60.325" x2="61.7825" y2="60.325" width="1.016" layer="16"/>
+<wire x1="59.055" y1="60.325" x2="56.515" y2="60.325" width="1.016" layer="16"/>
+<wire x1="52.07" y1="60.325" x2="54.61" y2="60.325" width="1.016" layer="16"/>
 <contactref element="IC6" pad="24"/>
+<wire x1="54.61" y1="60.325" x2="56.515" y2="60.325" width="1.016" layer="16"/>
+<wire x1="59.055" y1="60.325" x2="61.7825" y2="60.325" width="1.016" layer="16"/>
 <wire x1="99.695" y1="114.6175" x2="111.76" y2="114.6175" width="1.016" layer="16"/>
 <wire x1="111.76" y1="114.6175" x2="114.935" y2="114.6175" width="1.016" layer="16"/>
@@
 <wire x1="52.07" y1="86.36" x2="59.69" y2="86.36" width="0.6096" layer="16"/>
 <wire x1="59.69" y1="86.36" x2="60.8575" y2="87.5275" width="0.6096" layer="16"/>
-<wire x1="40.005" y1="60.325" x2="45.72" y2="60.325" width="0.8128" layer="16"/>
+<wire x1="40.005" y1="60.325" x2="46.99" y2="60.325" width="0.8128" layer="16"/>
 <contactref element="IC8" pad="20"/>
 <contactref element="IC9" pad="20"/>
 <contactref element="IC10" pad="20"/>
-<wire x1="45.72" y1="60.325" x2="52.07" y2="60.325" width="0.8128" layer="16"/>
+<wire x1="46.99" y1="60.325" x2="52.07" y2="60.325" width="0.8128" layer="16"/>
 <wire x1="131.4958" y1="84.455" x2="133.985" y2="84.455" width="0.6096" layer="16"/>
 <wire x1="133.985" y1="84.455" x2="133.985" y2="71.0692" width="0.6096" layer="16"/>
@@
 <wire x1="27.305" y1="49.315" x2="40.005" y2="49.315" width="0.8128" layer="16"/>
 <wire x1="40.005" y1="47.625" x2="40.005" y2="49.315" width="0.8128" layer="16"/>
-<wire x1="45.72" y1="60.325" x2="45.72" y2="50.8" width="0.8128" layer="16"/>
-<wire x1="45.72" y1="50.8" x2="44.235" y2="49.315" width="0.8128" layer="16"/>
-<wire x1="40.005" y1="49.315" x2="44.235" y2="49.315" width="0.8128" layer="16"/>
+<wire x1="46.99" y1="60.325" x2="46.99" y2="50.8" width="0.8128" layer="16"/>
+<wire x1="46.99" y1="50.8" x2="45.505" y2="49.315" width="0.8128" layer="16"/>
+<wire x1="40.005" y1="49.315" x2="45.505" y2="49.315" width="0.8128" layer="16"/>
 <contactref element="QG1" pad="14"/>
 <contactref element="R1" pad="1"/>
@@
 <wire x1="27.305" y1="47.625" x2="27.305" y2="49.315" width="0.8128" layer="16"/>
 <wire x1="8.255" y1="98.425" x2="8.255" y2="106.9975" width="1.016" layer="16"/>
+<contactref element="R2" pad="2"/>
+<wire x1="56.515" y1="59.4986" x2="56.515" y2="60.325" width="0.4064" layer="16"/>
+<contactref element="R3" pad="2"/>
+<wire x1="54.61" y1="57.785" x2="54.61" y2="60.325" width="0.6096" layer="16"/>
 </signal>
 <signal name="INT">
@@
 <wire x1="131.4958" y1="51.435" x2="126.365" y2="51.435" width="0.4064" layer="16"/>
 <contactref element="IC8" pad="1"/>
-<wire x1="131.4958" y1="51.435" x2="134.62" y2="51.435" width="0.4064" layer="16"/>
-<wire x1="134.62" y1="51.435" x2="135.89" y2="52.705" width="0.4064" layer="16"/>
-<wire x1="135.89" y1="52.705" x2="135.89" y2="82.55" width="0.4064" layer="16"/>
-<wire x1="135.89" y1="82.55" x2="137.795" y2="84.455" width="0.4064" layer="16"/>
-<wire x1="137.795" y1="84.455" x2="141.5542" y2="84.455" width="0.4064" layer="16"/>
+<wire x1="131.4958" y1="51.435" x2="134.3025" y2="51.435" width="0.4064" layer="16"/>
+<wire x1="134.3025" y1="51.435" x2="135.5725" y2="52.705" width="0.4064" layer="16"/>
+<wire x1="135.5725" y1="52.705" x2="135.5725" y2="82.55" width="0.4064" layer="16"/>
+<wire x1="135.5725" y1="82.55" x2="137.4775" y2="84.455" width="0.4064" layer="16"/>
+<wire x1="137.4775" y1="84.455" x2="141.5542" y2="84.455" width="0.4064" layer="16"/>
 </signal>
 <signal name="D1_IN">
@@
 <contactref element="IC2" pad="14"/>
 <contactref element="IC2" pad="13"/>
-<wire x1="59.055" y1="47.625" x2="62.23" y2="47.625" width="0.4064" layer="16"/>
-<wire x1="62.23" y1="47.625" x2="74.295" y2="47.625" width="0.4064" layer="16"/>
 <wire x1="59.055" y1="47.625" x2="59.055" y2="50.165" width="0.6096" layer="16"/>
 <wire x1="40.005" y1="37.465" x2="47.625" y2="37.465" width="0.4064" layer="16"/>
 <wire x1="47.625" y1="37.465" x2="48.895" y2="38.735" width="0.4064" layer="16"/>
-<wire x1="48.895" y1="38.735" x2="60.96" y2="38.735" width="0.4064" layer="16"/>
-<wire x1="60.96" y1="38.735" x2="62.23" y2="40.005" width="0.4064" layer="16"/>
-<wire x1="62.23" y1="40.005" x2="62.23" y2="47.625" width="0.4064" layer="16"/>
+<wire x1="48.895" y1="38.735" x2="61.595" y2="38.735" width="0.4064" layer="16"/>
+<via x="61.595" y="38.735" extent="1-16" drill="0.6" diameter="1.4224" shape="octagon"/>
+<wire x1="61.595" y1="38.735" x2="61.595" y2="47.625" width="0.4064" layer="1"/>
+<via x="61.595" y="47.625" extent="1-16" drill="0.6" diameter="1.4224" shape="octagon"/>
+<wire x1="59.69" y1="47.625" x2="61.595" y2="47.625" width="0.4064" layer="16"/>
+<wire x1="61.595" y1="47.625" x2="74.295" y2="47.625" width="0.4064" layer="16"/>
+<wire x1="59.69" y1="47.625" x2="59.055" y2="47.625" width="0" layer="19" extent="16-16"/>
 </signal>
 <signal name="N$30">
@@
 <wire x1="64.135" y1="65.405" x2="59.055" y2="65.405" width="0.4064" layer="16"/>
 </signal>
+<signal name="N$34">
+<contactref element="IC2" pad="25"/>
+<contactref element="IC2" pad="22"/>
+<contactref element="IC2" pad="16"/>
+<contactref element="R3" pad="1"/>
+<contactref element="IC2" pad="19"/>
+<wire x1="54.61" y1="42.545" x2="56.515" y2="42.545" width="0.6096" layer="16"/>
+<via x="56.515" y="42.545" extent="1-16" drill="0.6" diameter="1.4224" shape="octagon"/>
+<via x="56.515" y="34.925" extent="1-16" drill="0.6" diameter="1.4224" shape="octagon"/>
+<wire x1="56.515" y1="42.545" x2="59.055" y2="42.545" width="0.6096" layer="16"/>
+<wire x1="59.055" y1="42.545" x2="70.1675" y2="42.545" width="0.4064" layer="16"/>
+<wire x1="70.1675" y1="42.545" x2="74.295" y2="42.545" width="0.4064" layer="16"/>
+<wire x1="56.515" y1="42.545" x2="56.515" y2="34.925" width="0.4064" layer="1"/>
+<wire x1="56.515" y1="34.925" x2="59.055" y2="34.925" width="0.6096" layer="16"/>
+<wire x1="74.295" y1="34.925" x2="71.4375" y2="34.925" width="0.4064" layer="16"/>
+<wire x1="71.4375" y1="34.925" x2="70.1675" y2="36.195" width="0.4064" layer="16"/>
+<wire x1="70.1675" y1="36.195" x2="70.1675" y2="42.545" width="0.4064" layer="16"/>
+</signal>
+<signal name="N$36">
+<contactref element="IC2" pad="30"/>
+<contactref element="IC2" pad="29"/>
+<contactref element="IC2" pad="10"/>
+<contactref element="IC2" pad="11"/>
+<contactref element="R2" pad="1"/>
+<wire x1="56.515" y1="57.7986" x2="59.0414" y2="57.7986" width="0.6096" layer="16"/>
+<wire x1="59.0414" y1="57.7986" x2="59.055" y2="57.785" width="0.6096" layer="16"/>
+<wire x1="59.055" y1="55.245" x2="59.055" y2="57.785" width="0.6096" layer="16"/>
+<wire x1="59.055" y1="55.245" x2="74.295" y2="55.245" width="0.4064" layer="16"/>
+<wire x1="74.295" y1="52.705" x2="74.295" y2="55.245" width="0.6096" layer="16"/>
+</signal>
 </signals>

Commit message: IO board update (work in progress)
Parts:
- added R11, R4, R5: (no value), rcl:R0603
- added R6: (no value), rcl:0204/5
- moved C19 0.32 mm to (116.0, 65.4)
Connections:
- new net N$31: IC6.22, R5.1
- new net N$33: IC6.23, R4.1
- new net N$38: IC6.20, R6.1
- new net N$39: IC6.21, R11.1
- net VCC: now also R11.2, R4.2, R5.2, R6.2
Routing:
- net GND: track 138.2 -> 166.1 mm, vias 20 -> 22
- net VCC: track 643.0 -> 653.3 mm
- net N$38: track 0.00 -> 6.35 mm
- net N$39: track 0.00 -> 4.80 mm
- net N$33: track 0.00 -> 2.82 mm
- net N$31: track 0.00 -> 2.55 mm
Changed lines of the file:
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@@
 <setting verticaltext="up"/>
 </settings>
-<grid distance="25" unitdist="mil" unit="mil" style="lines" multiple="1" display="no" altdistance="12.5" altunitdist="mil" altunit="mil"/>
+<grid distance="25" unitdist="mil" unit="mil" style="lines" multiple="1" display="no" altdistance="1" altunitdist="mil" altunit="mil"/>
 <layers>
 <layer number="1" name="Top" color="4" fill="1" visible="yes" active="yes"/>
@@
 <element name="C16" library="rcl" package="C0603" value="100N" x="137.16" y="31.115" rot="MR0"/>
 <element name="C17" library="rcl" package="C0603" value="100N" x="128.0541" y="53.975" rot="MR0"/>
-<element name="C19" library="rcl" package="C0603" value="100N" x="116.3066" y="65.405" rot="MR0"/>
+<element name="C19" library="rcl" package="C0603" value="100N" x="115.9891" y="65.405" rot="MR0"/>
 <element name="JP3" library="pinhead" package="1X02/90" value="" x="4.445" y="108.2675" rot="R90"/>
 <element name="C21" library="rcl" package="E3,5-8" value="" x="8.255" y="96.647" rot="R270"/>
@@
 <element name="R2" library="rcl" package="R0603" value="" x="56.515" y="58.6486" rot="MR90"/>
 <element name="R3" library="rcl" package="0207/15" value="" x="54.61" y="50.165" rot="R90"/>
+<element name="R4" library="rcl" package="R0603" value="" x="121.92" y="63.119" rot="MR90"/>
+<element name="R5" library="rcl" package="R0603" value="" x="116.8391" y="61.1632" rot="MR90"/>
+<element name="R6" library="rcl" package="0204/5" value="" x="113.03" y="57.785" rot="R90"/>
+<element name="R11" library="rcl" package="R0603" value="" x="114.935" y="59.4868" rot="MR90"/>
 </elements>
 <signals>
@@
 <wire x1="94.615" y1="58.166" x2="94.615" y2="11.4935" width="0.6096" layer="1"/>
 <via x="94.615" y="11.4935" extent="1-16" drill="0.6" diameter="1.4224" shape="octagon"/>
+<via x="128.5875" y="59.69" extent="1-16" drill="0.6" diameter="1.4224" shape="octagon"/>
+<via x="128.5875" y="87.63" extent="1-16" drill="0.6" diameter="1.4224" shape="octagon"/>
+<wire x1="128.5875" y1="59.69" x2="128.5875" y2="87.63" width="0.6096" layer="1"/>
 </signal>
 <signal name="N$37">
@@
 <wire x1="121.92" y1="65.405" x2="121.92" y2="91.44" width="0.6096" layer="1"/>
 <via x="121.92" y="91.44" extent="1-16" drill="0.6" diameter="1.4224" shape="octagon"/>
-<wire x1="117.1566" y1="65.405" x2="119.38" y2="65.405" width="0.6096" layer="16"/>
+<wire x1="116.8391" y1="65.405" x2="119.38" y2="65.405" width="0.6096" layer="16"/>
 <contactref element="C30" pad="1"/>
 <wire x1="95.7825" y1="76.835" x2="97.4725" y2="76.835" width="0.6096" layer="16"/>
@@
 <contactref element="R3" pad="2"/>
 <wire x1="54.61" y1="57.785" x2="54.61" y2="60.325" width="0.6096" layer="16"/>
+<contactref element="R4" pad="2"/>
+<wire x1="121.92" y1="63.969" x2="121.92" y2="65.405" width="0.6096" layer="16"/>
+<contactref element="R5" pad="2"/>
+<wire x1="116.8391" y1="62.0132" x2="116.8391" y2="65.405" width="0.6096" layer="16"/>
+<contactref element="R11" pad="2"/>
+<contactref element="R6" pad="2"/>
+<wire x1="114.935" y1="60.3368" x2="114.935" y2="61.4172" width="0.6096" layer="16"/>
+<wire x1="114.935" y1="61.4172" x2="115.531" y2="62.0132" width="0.6096" layer="16"/>
+<wire x1="116.8391" y1="62.0132" x2="115.531" y2="62.0132" width="0.6096" layer="16"/>
+<wire x1="114.935" y1="60.3368" x2="113.0418" y2="60.3368" width="0.6096" layer="16"/>
+<wire x1="113.0418" y1="60.3368" x2="113.03" y2="60.325" width="0.6096" layer="16"/>
 </signal>
 <signal name="INT">
@@
 <contactref element="U$2" pad="6"/>
 <contactref element="IC10" pad="16"/>
-<wire x1="131.4958" y1="64.135" x2="123.825" y2="64.135" width="0.4064" layer="16"/>
 <via x="123.825" y="64.135" extent="1-16" drill="0.6" diameter="1.4224" shape="octagon"/>
 <wire x1="123.825" y1="64.135" x2="123.825" y2="26.035" width="0.4064" layer="1"/>
@@
 <wire x1="43.815" y1="67.945" x2="43.815" y2="26.035" width="0.4064" layer="1"/>
 <via x="43.815" y="26.035" extent="1-16" drill="0.6" diameter="1.4224" shape="octagon"/>
+<wire x1="131.4958" y1="64.135" x2="123.825" y2="64.135" width="0.4064" layer="16"/>
 </signal>
 <signal name="A3">
@@
 </signal>
 <signal name="A4">
-<via x="122.555" y="23.495" extent="1-16" drill="0.6" diameter="1.4224" shape="octagon"/>
+<via x="121.92" y="23.495" extent="1-16" drill="0.6" diameter="1.4224" shape="octagon"/>
 <contactref element="IC4" pad="13"/>
 <contactref element="IC10" pad="14"/>
-<via x="122.555" y="61.595" extent="1-16" drill="0.6" diameter="1.4224" shape="octagon"/>
-<wire x1="122.555" y1="61.595" x2="122.555" y2="23.495" width="0.4064" layer="1"/>
-<wire x1="131.4958" y1="61.595" x2="122.555" y2="61.595" width="0.4064" layer="16"/>
-<wire x1="122.555" y1="23.495" x2="130.175" y2="23.495" width="0.4064" layer="16"/>
+<via x="121.92" y="59.055" extent="1-16" drill="0.6" diameter="1.4224" shape="octagon"/>
+<wire x1="121.92" y1="59.055" x2="121.92" y2="23.495" width="0.4064" layer="1"/>
+<wire x1="121.92" y1="23.495" x2="130.175" y2="23.495" width="0.4064" layer="16"/>
 <wire x1="130.175" y1="23.495" x2="131.445" y2="24.765" width="0.4064" layer="16"/>
 <wire x1="131.445" y1="24.765" x2="133.985" y2="24.765" width="0.4064" layer="16"/>
 <wire x1="133.985" y1="24.765" x2="135.255" y2="23.495" width="0.4064" layer="16"/>
 <wire x1="135.255" y1="23.495" x2="140.335" y2="23.495" width="0.4064" layer="16"/>
+<wire x1="131.4958" y1="61.595" x2="124.46" y2="61.595" width="0.4064" layer="16"/>
+<wire x1="124.46" y1="61.595" x2="121.92" y2="59.055" width="0.4064" layer="16"/>
 </signal>
 <signal name="A5">
@@
 <via x="76.835" y="67.945" extent="1-16" drill="0.6" diameter="1.4224" shape="octagon"/>
 <wire x1="76.835" y1="67.945" x2="74.295" y2="67.945" width="0.4064" layer="16"/>
-<wire x1="133.985" y1="22.225" x2="121.92" y2="22.225" width="0.4064" layer="16"/>
-<wire x1="121.92" y1="22.225" x2="120.65" y2="23.495" width="0.4064" layer="16"/>
-<wire x1="120.65" y1="23.495" x2="76.835" y2="23.495" width="0.4064" layer="16"/>
+<wire x1="133.985" y1="22.225" x2="121.285" y2="22.225" width="0.4064" layer="16"/>
+<wire x1="121.285" y1="22.225" x2="120.015" y2="23.495" width="0.4064" layer="16"/>
+<wire x1="120.015" y1="23.495" x2="76.835" y2="23.495" width="0.4064" layer="16"/>
 </signal>
 <signal name="CF_CS0">
@@
 <wire x1="74.295" y1="52.705" x2="74.295" y2="55.245" width="0.6096" layer="16"/>
 </signal>
+<signal name="N$31">
+<contactref element="IC6" pad="22"/>
+<contactref element="R5" pad="1"/>
+<wire x1="116.8391" y1="60.3132" x2="119.3682" y2="60.3132" width="0.6096" layer="16"/>
+<wire x1="119.3682" y1="60.3132" x2="119.38" y2="60.325" width="0.6096" layer="16"/>
+</signal>
+<signal name="N$33">
+<contactref element="R4" pad="1"/>
+<contactref element="IC6" pad="23"/>
+<wire x1="119.38" y1="62.865" x2="120.2182" y2="62.865" width="0.6096" layer="16"/>
+<wire x1="120.2182" y1="62.865" x2="120.8532" y2="62.23" width="0.6096" layer="16"/>
+<wire x1="120.8532" y1="62.23" x2="121.881" y2="62.23" width="0.6096" layer="16"/>
+<wire x1="121.881" y1="62.23" x2="121.92" y2="62.269" width="0.6096" layer="16"/>
+</signal>
+<signal name="N$38">
+<contactref element="IC6" pad="20"/>
+<contactref element="R6" pad="1"/>
+<wire x1="113.03" y1="55.245" x2="119.38" y2="55.245" width="0.6096" layer="16"/>
+</signal>
+<signal name="N$39">
+<contactref element="IC6" pad="21"/>
+<contactref element="R11" pad="1"/>
+<wire x1="119.38" y1="57.785" x2="115.7868" y2="57.785" width="0.6096" layer="16"/>
+<wire x1="115.7868" y1="57.785" x2="114.935" y2="58.6368" width="0.6096" layer="16"/>
+</signal>
 </signals>

Commit message: IO board update
Parts:
- added JP1: (no value), pinhead:2X04
- added X4: 736880-49, con-conrad:736880-49
- moved C32 5.08 mm to (34.9, 50.2)
- moved IC11 5.08 mm to (31.1, 40.0)
- moved QG1 5.08 mm to (18.4, 40.0)
- moved R1 5.08 mm to (18.4, 47.6)
- moved C31 5.08 mm to (22.2, 50.2)
Connections:
- net N$27 renamed BAUDRATE_38400
- new net BAUDRATE_153600: IC11.4
- new net BAUDRATE_19200: IC11.11, JP1.1
- new net BAUDRATE_2400: IC11.8, JP1.7
- new net BAUDRATE_307200: IC11.3
- new net BAUDRATE_4800: IC11.9, JP1.5
- new net BAUDRATE_76800: IC11.5
- new net BAUDRATE_9600: IC11.10, IC2.27, JP1.3
- net BAUDRATE: now also JP1.2, JP1.4, JP1.6, JP1.8; no longer IC11.10, IC2.27
Routing:
- net BAUDRATE_9600: track 0.00 -> 45.1 mm
- net BAUDRATE: track 48.2 -> 39.0 mm
- net BAUDRATE_4800: track 0.00 -> 3.18 mm
- net BAUDRATE_2400: track 0.00 -> 3.18 mm
- net BAUDRATE_19200: track 0.00 -> 3.18 mm
- net VCC: track 653.3 -> 656.3 mm
