File: hardware/IO_board/IO.sch (EAGLE design)
At the start: 52 parts, among them IC1 MAX232, IC4 74HCT139N, IC5 74AC06N, IC7 MAX232, J1 DIN5, X2 CRYSTALS-NOGND-CFPX-217

Commit message: CPU board and I/O board update
Parts:
- added IC10, IC8, IC9: 74HCT245DW, 74xx-eu:74HCT245DW
- R7: device rcl:R-EU_0204/5 -> rcl:R-EU_0204/7
Connections:
- new net !IORQ_IN: IC9A.A7, SV2.44
- new net A0_IN: IC10A.A1, SV2.15
- new net A1_IN: IC10A.A2, SV2.16
- new net A2_IN: IC10A.A3, SV2.17
- new net A3_IN: IC10A.A4, SV2.18
- new net A4_IN: IC10A.A5, SV2.19
- new net CLK_IN: IC9A.A3, SV2.36
- new net D0_IN: IC8A.A1, SV2.7
- new net D1_IN: IC8A.A2, SV2.8
- new net D2_IN: IC8A.A3, SV2.9
- new net D3_IN: IC8A.A4, SV2.10
- new net D4_IN: IC8A.A5, SV2.11
- new net D5_IN: IC8A.A6, SV2.12
- new net D6_IN: IC8A.A7, SV2.13
- new net D7_IN: IC8A.A8, SV2.14
- new net M1_IN: IC9A.A8, SV2.43
- new net RD_IN: IC9A.A1, SV2.34
- new net WR_IN: IC9A.A2, SV2.35
- net !IORQ: now also IC9A.B7; no longer SV2.44
- net A0: now also IC10A.B1; no longer SV2.15
- net A1: now also IC10A.B2; no longer SV2.16
- net A2: now also IC10A.B3; no longer SV2.17
- net A3: now also IC10A.B4; no longer SV2.18
- net A4: now also IC10A.B5; no longer SV2.19
- net CLK: now also IC9A.B3; no longer SV2.36
- net D0: now also IC8A.B1; no longer SV2.7
- net D1: now also IC8A.B2; no longer SV2.8
- net D2: now also IC8A.B3; no longer SV2.9
- net D3: now also IC8A.B4; no longer SV2.10
- net D4: now also IC8A.B5; no longer SV2.11
- net D5: now also IC8A.B6; no longer SV2.12
- net D6: now also IC8A.B7; no longer SV2.13
- net D7: now also IC8A.B8; no longer SV2.14
- net GND: now also IC10A.A6, IC10A.A7, IC10A.A8, IC10A.G, IC8A.G, IC9A.A4, IC9A.A5, IC9A.A6, IC9A.G
- net M1: now also IC9A.B8; no longer SV2.43
- net RD: now also IC8A.DIR, IC9A.B1; no longer SV2.34
- net WR: now also IC9A.B2; no longer SV2.35

Commit message: I/O board updated (work in progress)
Parts:
- added C30, C31, C32: 100N, rcl:C-EUC0603
- added IC11: 74HCT393N, 74xx-eu:74HCT393N
- added QG1: (no value), crystal:XO-14
- added R1: (no value), rcl:R-EU_R0603
Connections:
- new net BAUDRATE: IC11B.QB, IC2.RXCA, IC2.RXTXCB, IC2.TXCA
- new net N$26: IC11A.A, QG1.OUT
- new net N$27: IC11A.QD, IC11B.A
- new net N$30: QG1.TS, R1.2
- new net N$32: IC2.IEO, IC6.IEI
- net A4: no longer IC4A.A
- net CS_1: no longer IC4A.G
- net GND: now also C30.2, C31.2, C32.2, IC11A.CLR, IC11B.CLR, IC11P.GND, IC4A.A, IC4A.G, IC5C.I, QG1.GND
- net TIMER_CS: now also IC6.CE
- net UART_CS: now also IC2.CE
- net VCC: now also C30.1, C31.1, C32.1, IC10A.DIR, IC11P.VCC, IC9A.DIR, QG1.VCC, R1.1
Other:
- moved on the sheet: C1, C10, C12, C14, C15, C16, C17, C19, C2, C21, C24, C28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

Commit message: IO board update (work in progress)
Parts:
- added R2: (no value), rcl:R-EU_R0603
- added R3: (no value), rcl:R-EU_0207/15
Connections:
- new net N$34: IC2.DCDA, IC2.DCDB, IC2.DTRA, IC2.DTRB, R3.1
- new net N$36: IC2.RIA, IC2.RIB, IC2.W/RDYA, IC2.W/RDYB, R2.1
- net VCC: now also R2.2, R3.2
Changed lines of the file:
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@@
 <part name="R1" library="rcl" deviceset="R-EU_" device="R0603"/>
 <part name="GND16" library="supply1" deviceset="GND" device=""/>
+<part name="R2" library="rcl" deviceset="R-EU_" device="R0603"/>
+<part name="R3" library="rcl" deviceset="R-EU_" device="0207/15"/>
 </parts>
 <sheets>
@@
 <instance part="R1" gate="G$1" x="172.72" y="314.96" rot="R270"/>
 <instance part="GND16" gate="1" x="142.24" y="292.1"/>
+<instance part="R2" gate="G$1" x="86.36" y="246.38" rot="R90"/>
+<instance part="R3" gate="G$1" x="109.22" y="233.68" rot="R90"/>
 </instances>
 <busses>
@@
 <label x="142.24" y="325.12" size="1.4224" layer="95" rot="R90" xref="yes"/>
 </segment>
+<segment>
+<pinref part="R2" gate="G$1" pin="2"/>
+<wire x1="86.36" y1="251.46" x2="86.36" y2="254" width="0.1524" layer="91"/>
+</segment>
+<segment>
+<pinref part="R3" gate="G$1" pin="2"/>
+<wire x1="109.22" y1="238.76" x2="109.22" y2="241.3" width="0.1524" layer="91"/>
+</segment>
 </net>
 <net name="N$15" class="0">
@@
 <segment>
 <pinref part="IC2" gate="G$1" pin="TXDB"/>
-<wire x1="81.28" y1="205.74" x2="86.36" y2="205.74" width="0.1524" layer="91"/>
-<label x="86.36" y="205.74" size="1.4224" layer="95" xref="yes"/>
+<wire x1="81.28" y1="205.74" x2="91.44" y2="205.74" width="0.1524" layer="91"/>
+<label x="91.44" y="205.74" size="1.4224" layer="95" xref="yes"/>
 </segment>
 </net>
@@
 <segment>
 <pinref part="IC2" gate="G$1" pin="RXDB"/>
-<wire x1="81.28" y1="208.28" x2="86.36" y2="208.28" width="0.1524" layer="91"/>
-<label x="86.36" y="208.28" size="1.4224" layer="95" xref="yes"/>
+<wire x1="81.28" y1="208.28" x2="91.44" y2="208.28" width="0.1524" layer="91"/>
+<label x="91.44" y="208.28" size="1.4224" layer="95" xref="yes"/>
 </segment>
 </net>
@@
 <segment>
 <pinref part="IC2" gate="G$1" pin="RXTXCB"/>
-<wire x1="81.28" y1="203.2" x2="86.36" y2="203.2" width="0.1524" layer="91"/>
-<label x="86.36" y="203.2" size="1.4224" layer="95" xref="yes"/>
+<wire x1="81.28" y1="203.2" x2="91.44" y2="203.2" width="0.1524" layer="91"/>
+<label x="91.44" y="203.2" size="1.4224" layer="95" xref="yes"/>
 </segment>
 <segment>
@@
 </segment>
 </net>
+<net name="N$34" class="0">
+<segment>
+<pinref part="IC2" gate="G$1" pin="DCDB"/>
+<pinref part="IC2" gate="G$1" pin="DTRB"/>
+<wire x1="83.82" y1="187.96" x2="81.28" y2="187.96" width="0.1524" layer="91"/>
+<wire x1="83.82" y1="187.96" x2="83.82" y2="185.42" width="0.1524" layer="91"/>
+<wire x1="83.82" y1="185.42" x2="81.28" y2="185.42" width="0.1524" layer="91"/>
+<pinref part="IC2" gate="G$1" pin="DTRA"/>
+<wire x1="81.28" y1="215.9" x2="83.82" y2="215.9" width="0.1524" layer="91"/>
+<wire x1="83.82" y1="215.9" x2="109.22" y2="215.9" width="0.1524" layer="91"/>
+<wire x1="109.22" y1="215.9" x2="109.22" y2="228.6" width="0.1524" layer="91"/>
+<pinref part="R3" gate="G$1" pin="1"/>
+<pinref part="IC2" gate="G$1" pin="DCDA"/>
+<wire x1="81.28" y1="213.36" x2="83.82" y2="213.36" width="0.1524" layer="91"/>
+<wire x1="83.82" y1="213.36" x2="83.82" y2="215.9" width="0.1524" layer="91"/>
+<junction x="83.82" y="215.9"/>
+<wire x1="83.82" y1="187.96" x2="83.82" y2="213.36" width="0.1524" layer="91"/>
+<junction x="83.82" y="187.96"/>
+<junction x="83.82" y="213.36"/>
+</segment>
+</net>
+<net name="N$36" class="0">
+<segment>
+<pinref part="IC2" gate="G$1" pin="RIB"/>
+<pinref part="IC2" gate="G$1" pin="W/RDYB"/>
+<wire x1="86.36" y1="200.66" x2="81.28" y2="200.66" width="0.1524" layer="91"/>
+<wire x1="86.36" y1="200.66" x2="86.36" y2="195.58" width="0.1524" layer="91"/>
+<wire x1="86.36" y1="195.58" x2="81.28" y2="195.58" width="0.1524" layer="91"/>
+<pinref part="IC2" gate="G$1" pin="W/RDYA"/>
+<pinref part="R2" gate="G$1" pin="1"/>
+<wire x1="81.28" y1="228.6" x2="86.36" y2="228.6" width="0.1524" layer="91"/>
+<wire x1="86.36" y1="228.6" x2="86.36" y2="241.3" width="0.1524" layer="91"/>
+<pinref part="IC2" gate="G$1" pin="RIA"/>
+<wire x1="81.28" y1="223.52" x2="86.36" y2="223.52" width="0.1524" layer="91"/>
+<wire x1="86.36" y1="223.52" x2="86.36" y2="228.6" width="0.1524" layer="91"/>
+<junction x="86.36" y="228.6"/>
+<wire x1="86.36" y1="200.66" x2="86.36" y2="223.52" width="0.1524" layer="91"/>
+<junction x="86.36" y="200.66"/>
+<junction x="86.36" y="223.52"/>
+</segment>
+</net>

Commit message: IO board update (work in progress)
Parts:
- added R11, R4, R5: (no value), rcl:R-EU_R0603
- added R6: (no value), rcl:R-EU_0204/5
Connections:
- new net N$31: IC6.TRG1, R5.1
- new net N$33: IC6.TRG0, R4.1
- new net N$38: IC6.TRG3, R6.1
- new net N$39: IC6.TRG2, R11.1
- net VCC: now also R11.2, R4.2, R5.2, R6.2
Changed lines of the file:
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@@
 <part name="R2" library="rcl" deviceset="R-EU_" device="R0603"/>
 <part name="R3" library="rcl" deviceset="R-EU_" device="0207/15"/>
+<part name="R4" library="rcl" deviceset="R-EU_" device="R0603"/>
+<part name="R5" library="rcl" deviceset="R-EU_" device="R0603"/>
+<part name="R6" library="rcl" deviceset="R-EU_" device="0204/5"/>
+<part name="R11" library="rcl" deviceset="R-EU_" device="R0603"/>
 </parts>
 <sheets>
@@
 <instance part="R2" gate="G$1" x="86.36" y="246.38" rot="R90"/>
 <instance part="R3" gate="G$1" x="109.22" y="233.68" rot="R90"/>
+<instance part="R4" gate="G$1" x="83.82" y="332.74" rot="R90"/>
+<instance part="R5" gate="G$1" x="88.9" y="332.74" rot="R90"/>
+<instance part="R6" gate="G$1" x="99.06" y="332.74" rot="R90"/>
+<instance part="R11" gate="G$1" x="93.98" y="332.74" rot="R90"/>
 </instances>
 <busses>
@@
 </segment>
 <segment>
+<pinref part="GND5" gate="1" pin="GND"/>
 <pinref part="IC6" gate="1" pin="GND"/>
 <wire x1="81.28" y1="281.94" x2="83.82" y2="281.94" width="0.1524" layer="91"/>
-<pinref part="GND5" gate="1" pin="GND"/>
 <wire x1="83.82" y1="281.94" x2="83.82" y2="279.4" width="0.1524" layer="91"/>
 </segment>
@@
 <wire x1="109.22" y1="238.76" x2="109.22" y2="241.3" width="0.1524" layer="91"/>
 </segment>
+<segment>
+<pinref part="R4" gate="G$1" pin="2"/>
+<wire x1="83.82" y1="337.82" x2="83.82" y2="340.36" width="0.1524" layer="91"/>
+<pinref part="R5" gate="G$1" pin="2"/>
+<wire x1="83.82" y1="340.36" x2="88.9" y2="340.36" width="0.1524" layer="91"/>
+<wire x1="88.9" y1="340.36" x2="88.9" y2="337.82" width="0.1524" layer="91"/>
+<wire x1="88.9" y1="340.36" x2="93.98" y2="340.36" width="0.1524" layer="91"/>
+<junction x="88.9" y="340.36"/>
+<wire x1="93.98" y1="340.36" x2="99.06" y2="340.36" width="0.1524" layer="91"/>
+<wire x1="88.9" y1="340.36" x2="88.9" y2="342.9" width="0.1524" layer="91"/>
+<pinref part="R11" gate="G$1" pin="2"/>
+<wire x1="93.98" y1="337.82" x2="93.98" y2="340.36" width="0.1524" layer="91"/>
+<junction x="93.98" y="340.36"/>
+<pinref part="R6" gate="G$1" pin="2"/>
+<wire x1="99.06" y1="340.36" x2="99.06" y2="337.82" width="0.1524" layer="91"/>
+</segment>
 </net>
 <net name="N$15" class="0">
@@
 </segment>
 </net>
+<net name="N$31" class="0">
+<segment>
+<pinref part="IC6" gate="1" pin="TRG1"/>
+<pinref part="R5" gate="G$1" pin="1"/>
+<wire x1="81.28" y1="317.5" x2="88.9" y2="317.5" width="0.1524" layer="91"/>
+<wire x1="88.9" y1="317.5" x2="88.9" y2="327.66" width="0.1524" layer="91"/>
+</segment>
+</net>
+<net name="N$33" class="0">
+<segment>
+<pinref part="R4" gate="G$1" pin="1"/>
+<wire x1="83.82" y1="325.12" x2="83.82" y2="327.66" width="0.1524" layer="91"/>
+<pinref part="IC6" gate="1" pin="TRG0"/>
+<wire x1="81.28" y1="325.12" x2="83.82" y2="325.12" width="0.1524" layer="91"/>
+</segment>
+</net>
+<net name="N$38" class="0">
+<segment>
+<pinref part="IC6" gate="1" pin="TRG3"/>
+<pinref part="R6" gate="G$1" pin="1"/>
+<wire x1="81.28" y1="302.26" x2="99.06" y2="302.26" width="0.1524" layer="91"/>
+<wire x1="99.06" y1="302.26" x2="99.06" y2="327.66" width="0.1524" layer="91"/>
+</segment>
+</net>
+<net name="N$39" class="0">
+<segment>
+<pinref part="IC6" gate="1" pin="TRG2"/>
+<wire x1="81.28" y1="309.88" x2="93.98" y2="309.88" width="0.1524" layer="91"/>
+<pinref part="R11" gate="G$1" pin="1"/>
+<wire x1="93.98" y1="327.66" x2="93.98" y2="309.88" width="0.1524" layer="91"/>
+</segment>
+</net>

Commit message: IO board update
Parts:
- added JP1: (no value), pinhead:PINHD-2X4
- added X4: 736880-49, con-conrad:736880-49
Connections:
- net N$27 renamed BAUDRATE_38400
- new net BAUDRATE_153600: IC11A.QB
- new net BAUDRATE_19200: IC11B.QA, JP1.1
- new net BAUDRATE_2400: IC11B.QD, JP1.7
- new net BAUDRATE_307200: IC11A.QA
- new net BAUDRATE_4800: IC11B.QC, JP1.5
- new net BAUDRATE_76800: IC11A.QC
- new net BAUDRATE_9600: IC11B.QB, IC2.RXTXCB, JP1.3
- net BAUDRATE: now also JP1.2, JP1.4, JP1.6, JP1.8; no longer IC11B.QB, IC2.RXTXCB
Changed lines of the file:
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@@
 <layer number="154" name="FabDoc2" color="7" fill="1" visible="yes" active="yes"/>
 <layer number="155" name="FabDoc3" color="7" fill="1" visible="yes" active="yes"/>
+<layer number="156" name="gesam-Maß" color="1" fill="7" visible="no" active="no"/>
+<layer number="157" name="FaceMchng" color="3" fill="1" visible="no" active="no"/>
+<layer number="158" name="FaceMMeas" color="3" fill="1" visible="no" active="no"/>
+<layer number="159" name="Geh-Bear2" color="1" fill="7" visible="no" active="no"/>
+<layer number="160" name="Topologie" color="9" fill="1" visible="no" active="no"/>
+<layer number="161" name="tomplace2" color="7" fill="1" visible="no" active="no"/>
 <layer number="191" name="mNets" color="7" fill="1" visible="yes" active="yes"/>
 <layer number="192" name="mBusses" color="7" fill="1" visible="yes" active="yes"/>
@@
 <layer number="250" name="Descript" color="3" fill="1" visible="no" active="no"/>
 <layer number="251" name="SMDround" color="12" fill="11" visible="no" active="no"/>
+<layer number="252" name="BR-BS" color="7" fill="1" visible="no" active="no"/>
+<layer number="253" name="BR-LS" color="7" fill="1" visible="no" active="no"/>
 <layer number="254" name="cooling" color="7" fill="1" visible="yes" active="yes"/>
 <layer number="255" name="HELP" color="7" fill="1" visible="yes" active="yes"/>
@@
 <part name="R6" library="rcl" deviceset="R-EU_" device="0204/5"/>
 <part name="R11" library="rcl" deviceset="R-EU_" device="R0603"/>
+<part name="X4" library="con-conrad" deviceset="736880-49" device=""/>
+<part name="JP1" library="pinhead" deviceset="PINHD-2X4" device=""/>
 </parts>
 <sheets>
@@
 <instance part="R6" gate="G$1" x="99.06" y="332.74" rot="R90"/>
 <instance part="R11" gate="G$1" x="93.98" y="332.74" rot="R90"/>
+<instance part="X4" gate="G$1" x="73.66" y="363.22" rot="MR0"/>
+<instance part="JP1" gate="A" x="269.24" y="271.78"/>
 </instances>
 <busses>
@@
 </segment>
 </net>
-<net name="N$27" class="0">
+<net name="BAUDRATE_38400" class="0">
 <segment>
 <pinref part="IC11" gate="B" pin="A"/>
@@
 <pinref part="IC11" gate="A" pin="QD"/>
 <wire x1="205.74" y1="294.64" x2="203.2" y2="294.64" width="0.1524" layer="91"/>
+<wire x1="205.74" y1="294.64" x2="210.82" y2="294.64" width="0.1524" layer="91"/>
+<junction x="205.74" y="294.64"/>
+<label x="210.82" y="294.64" size="1.4224" layer="95" xref="yes"/>
 </segment>
 </net>
 <net name="BAUDRATE" class="0">
-<segment>
-<pinref part="IC11" gate="B" pin="QB"/>
-<wire x1="203.2" y1="274.32" x2="210.82" y2="274.32" width="0.1524" layer="91"/>
-<label x="210.82" y="274.32" size="1.4224" layer="95" xref="yes"/>
-</segment>
-<segment>
-<pinref part="IC2" gate="G$1" pin="RXTXCB"/>
-<wire x1="81.28" y1="203.2" x2="91.44" y2="203.2" width="0.1524" layer="91"/>
-<label x="91.44" y="203.2" size="1.4224" layer="95" xref="yes"/>
-</segment>
 <segment>
 <pinref part="IC2" gate="G$1" pin="TXCA"/>
@@
 <wire x1="81.28" y1="236.22" x2="88.9" y2="236.22" width="0.1524" layer="91"/>
 <label x="88.9" y="236.22" size="1.4224" layer="95" xref="yes"/>
+</segment>
+<segment>
+<pinref part="JP1" gate="A" pin="2"/>
+<wire x1="274.32" y1="276.86" x2="281.94" y2="276.86" width="0.1524" layer="91"/>
+<wire x1="281.94" y1="276.86" x2="281.94" y2="274.32" width="0.1524" layer="91"/>
+<wire x1="281.94" y1="274.32" x2="281.94" y2="271.78" width="0.1524" layer="91"/>
+<wire x1="281.94" y1="271.78" x2="281.94" y2="269.24" width="0.1524" layer="91"/>
+<wire x1="281.94" y1="269.24" x2="274.32" y2="269.24" width="0.1524" layer="91"/>
+<pinref part="JP1" gate="A" pin="8"/>
+<pinref part="JP1" gate="A" pin="4"/>
+<wire x1="274.32" y1="274.32" x2="281.94" y2="274.32" width="0.1524" layer="91"/>
+<junction x="281.94" y="274.32"/>
+<pinref part="JP1" gate="A" pin="6"/>
+<wire x1="274.32" y1="271.78" x2="281.94" y2="271.78" width="0.1524" layer="91"/>
+<junction x="281.94" y="271.78"/>
+<wire x1="281.94" y1="271.78" x2="287.02" y2="271.78" width="0.1524" layer="91"/>
 </segment>
 </net>
@@
 </segment>
 </net>
+<net name="BAUDRATE_9600" class="0">
+<segment>
+<pinref part="IC11" gate="B" pin="QB"/>
+<wire x1="203.2" y1="274.32" x2="210.82" y2="274.32" width="0.1524" layer="91"/>
+<label x="210.82" y="274.32" size="1.4224" layer="95" xref="yes"/>
+</segment>
+<segment>
+<pinref part="JP1" gate="A" pin="3"/>
+<wire x1="266.7" y1="274.32" x2="256.54" y2="274.32" width="0.1524" layer="91"/>
+<label x="256.54" y="274.32" size="1.4224" layer="95" rot="R180" xref="yes"/>
+</segment>
+<segment>
+<pinref part="IC2" gate="G$1" pin="RXTXCB"/>
+<wire x1="81.28" y1="203.2" x2="91.44" y2="203.2" width="0.1524" layer="91"/>
+<label x="91.44" y="203.2" size="1.4224" layer="95" xref="yes"/>
+</segment>
+</net>
+<net name="BAUDRATE_4800" class="0">
+<segment>
+<pinref part="IC11" gate="B" pin="QC"/>
+<wire x1="203.2" y1="271.78" x2="210.82" y2="271.78" width="0.1524" layer="91"/>
+<label x="210.82" y="271.78" size="1.4224" layer="95" xref="yes"/>
+</segment>
+<segment>
+<pinref part="JP1" gate="A" pin="5"/>
+<wire x1="266.7" y1="271.78" x2="256.54" y2="271.78" width="0.1524" layer="91"/>
+<label x="256.54" y="271.78" size="1.4224" layer="95" rot="R180" xref="yes"/>
+</segment>
+</net>
+<net name="BAUDRATE_2400" class="0">
+<segment>
+<pinref part="IC11" gate="B" pin="QD"/>
+<wire x1="203.2" y1="269.24" x2="210.82" y2="269.24" width="0.1524" layer="91"/>
+<label x="210.82" y="269.24" size="1.4224" layer="95" xref="yes"/>
+</segment>
+<segment>
+<pinref part="JP1" gate="A" pin="7"/>
+<wire x1="266.7" y1="269.24" x2="256.54" y2="269.24" width="0.1524" layer="91"/>
+<label x="256.54" y="269.24" size="1.4224" layer="95" rot="R180" xref="yes"/>
+</segment>
+</net>
+<net name="BAUDRATE_19200" class="0">
+<segment>
+<pinref part="IC11" gate="B" pin="QA"/>
+<wire x1="203.2" y1="276.86" x2="210.82" y2="276.86" width="0.1524" layer="91"/>
+<label x="210.82" y="276.86" size="1.4224" layer="95" xref="yes"/>
+</segment>
+<segment>
+<pinref part="JP1" gate="A" pin="1"/>
+<wire x1="266.7" y1="276.86" x2="256.54" y2="276.86" width="0.1524" layer="91"/>
+<label x="256.54" y="276.86" size="1.4224" layer="95" rot="R180" xref="yes"/>
+</segment>
+</net>
+<net name="BAUDRATE_76800" class="0">
+<segment>
+<pinref part="IC11" gate="A" pin="QC"/>
+<wire x1="203.2" y1="297.18" x2="210.82" y2="297.18" width="0.1524" layer="91"/>
+<label x="210.82" y="297.18" size="1.4224" layer="95" xref="yes"/>
+</segment>
+</net>
+<net name="BAUDRATE_153600" class="0">
+<segment>
+<pinref part="IC11" gate="A" pin="QB"/>
+<wire x1="203.2" y1="299.72" x2="210.82" y2="299.72" width="0.1524" layer="91"/>
+<label x="210.82" y="299.72" size="1.4224" layer="95" xref="yes"/>
+</segment>
+</net>
+<net name="BAUDRATE_307200" class="0">
+<segment>
+<pinref part="IC11" gate="A" pin="QA"/>
+<wire x1="203.2" y1="302.26" x2="210.82" y2="302.26" width="0.1524" layer="91"/>
+<label x="210.82" y="302.26" size="1.4224" layer="95" xref="yes"/>
+</segment>
+</net>

Commit message: CPU and I/O board update
Parts:
- removed IC11: 74HCT393N, 74xx-eu:74HCT393N
- removed JP1: (no value), pinhead:PINHD-2X4
- removed QG1: (no value), crystal:XO-14
- R1: device rcl:R-EU_R0603 -> rcl:R-EU_0204/7
Connections:
- removed net 8275_DACK: SV2.2
- removed net BAUDRATE: IC2.RXCA, IC2.TXCA, JP1.2, JP1.4, JP1.6, JP1.8
- removed net BAUDRATE_153600: IC11A.QB
- removed net BAUDRATE_19200: IC11B.QA, JP1.1
- removed net BAUDRATE_2400: IC11B.QD, JP1.7
- removed net BAUDRATE_307200: IC11A.QA
- removed net BAUDRATE_38400: IC11A.QD, IC11B.A
- removed net BAUDRATE_4800: IC11B.QC, JP1.5
- removed net BAUDRATE_76800: IC11A.QC
- removed net BAUDRATE_9600: IC11B.QB, IC2.RXTXCB, JP1.3
- removed net N$26: IC11A.A, QG1.OUT
- removed net N$30: QG1.TS, R1.2
- removed net RDYIN: SV2.1
- new net BAUDRATE_A: IC2.RXCA, IC2.TXCA, IC6.TO1
- new net BAUDRATE_B: IC2.RXTXCB, IC6.TO2
- new net BOARD_ENABLE: IC8A.G
- new net IEI: IC2.IEI, SV2.1
- new net IEO: IC6.IEO, SV2.2
- new net TO0: IC6.TO0, R1.1
- net GND: no longer IC11A.CLR, IC11B.CLR, IC11P.GND, IC8A.G, QG1.GND
- net VCC: no longer IC11P.VCC, QG1.VCC, R1.1
Other:
- moved on the sheet: R1
