File: hardware/IO_board/IO.sch (EAGLE design)
At the start: 73 parts, among them IC1 MAX232, IC10 74HCT245DW, IC11 74LVC1G08DBV, IC4 74HCT139N, IC5 74AC06N, IC7 MAX232, IC8 74HCT245DW, IC9 74HCT245DW, J1 DIN5, T1 BC847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

Commit message: Separate baudrate generator on I/O board
Parts:
- added C36, C37: 100N, rcl:C-EUC0603
- added IC12: 74HCT393N, 74xx-eu:74HCT393N
- added JP1: (no value), pinhead:PINHD-2X5
- added QG1: (no value), crystal:XO-14
- added R12: (no value), rcl:R-EU_R0603
- R3: device rcl:R-EU_0207/15 -> rcl:R-EU_0204/5
Connections:
- removed net BAUDRATE_A: IC2.RXCA, IC2.TXCA, IC6.TO1
- new net 1228800HZ: IC12B.QA, JP1.3
- new net 153600HZ: IC12B.QD, IC2.RXCA, IC2.TXCA, JP1.9
- new net 2457600HZ: IC12B.A, JP1.1, QG1.OUT
- new net 307200HZ: IC12B.QC, JP1.7
- new net 614400HZ: IC12B.QB, JP1.5
- net A0: now also IC6.CS0
- net A1: now also IC6.CS1
- net BAUDRATE_B: now also JP1.10, JP1.2, JP1.4, JP1.6, JP1.8; no longer IC6.TO2
- net GND: now also C36.2, C37.2, IC12A.A, IC12A.CLR, IC12B.CLR, IC12P.GND, IC2.DCDA, IC2.DCDB, QG1.GND
- net IEI: now also R3.1
- net N$34: now also QG1.TS, R12.2; no longer IC2.DCDA, IC2.DCDB, IC2.DTRA, IC2.DTRB, R3.1
- net N$36: no longer IC2.W/RDYA, IC2.W/RDYB
- net VCC: now also C36.1, C37.1, IC12P.VCC, QG1.VCC, R12.1
Other:
- moved on the sheet: C1, C10, C12, C14, C15, C16, C17, C19, C2, C21, C24, C28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

Commit message: I/O board: 0R resistors added to set baudrate at DART channel A
Parts:
- added R13: (no value), rcl:R-EU_R0603
- added R16, R17, R18, R20, R21: 0R, rcl:R-EU_R0603
Connections:
- new net BAUDRATE_A: IC2.RXCA, IC2.TXCA, R16.2, R17.2, R18.2, R20.2, R21.2
- new net N$41: IC12A.CLR, R13.2
- net 1228800HZ: now also R17.1
- net 153600HZ: now also R21.1; no longer IC2.RXCA, IC2.TXCA
- net 2457600HZ: now also R16.1
- net 307200HZ: now also R20.1
- net 614400HZ: now also R18.1
- net GND: no longer IC12A.CLR
- net VCC: now also IC2.VCC, R13.1
Other:
- moved on the sheet: IC12A
Changed lines of the file:
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@@
 <part name="C37" library="rcl" deviceset="C-EU" device="C0603" value="100N"/>
 <part name="R12" library="rcl" deviceset="R-EU_" device="R0603"/>
+<part name="R13" library="rcl" deviceset="R-EU_" device="R0603"/>
+<part name="R17" library="rcl" deviceset="R-EU_" device="R0603" value="0R"/>
+<part name="R18" library="rcl" deviceset="R-EU_" device="R0603" value="0R"/>
+<part name="R20" library="rcl" deviceset="R-EU_" device="R0603" value="0R"/>
+<part name="R21" library="rcl" deviceset="R-EU_" device="R0603" value="0R"/>
+<part name="R16" library="rcl" deviceset="R-EU_" device="R0603" value="0R"/>
 </parts>
 <sheets>
@@
 <instance part="GND13" gate="1" x="83.82" y="172.72"/>
 <instance part="R3" gate="G$1" x="43.18" y="246.38" rot="R90"/>
-<instance part="IC12" gate="A" x="-233.68" y="88.9"/>
+<instance part="IC12" gate="A" x="-226.06" y="88.9"/>
 <instance part="IC12" gate="B" x="-233.68" y="66.04"/>
 <instance part="GND25" gate="1" x="-248.92" y="55.88"/>
@@
 <instance part="C37" gate="G$1" x="-73.66" y="228.6"/>
 <instance part="R12" gate="G$1" x="-254" y="81.28" rot="R270"/>
+<instance part="R13" gate="G$1" x="-241.3" y="99.06" rot="R270"/>
+<instance part="R17" gate="G$1" x="-203.2" y="10.16"/>
+<instance part="R18" gate="G$1" x="-203.2" y="2.54"/>
+<instance part="R20" gate="G$1" x="-203.2" y="-5.08"/>
+<instance part="R21" gate="G$1" x="-203.2" y="-12.7"/>
+<instance part="R16" gate="G$1" x="-203.2" y="17.78"/>
 </instances>
 <busses>
@@
 <wire x1="-246.38" y1="60.96" x2="-248.92" y2="60.96" width="0.1524" layer="91"/>
 <wire x1="-248.92" y1="60.96" x2="-248.92" y2="58.42" width="0.1524" layer="91"/>
-<pinref part="IC12" gate="A" pin="CLR"/>
-<wire x1="-246.38" y1="83.82" x2="-248.92" y2="83.82" width="0.1524" layer="91"/>
-<wire x1="-248.92" y1="83.82" x2="-248.92" y2="60.96" width="0.1524" layer="91"/>
+<wire x1="-248.92" y1="91.44" x2="-248.92" y2="60.96" width="0.1524" layer="91"/>
 <junction x="-248.92" y="60.96"/>
 <pinref part="IC12" gate="A" pin="A"/>
-<wire x1="-246.38" y1="91.44" x2="-248.92" y2="91.44" width="0.1524" layer="91"/>
-<wire x1="-248.92" y1="91.44" x2="-248.92" y2="83.82" width="0.1524" layer="91"/>
-<junction x="-248.92" y="83.82"/>
+<wire x1="-238.76" y1="91.44" x2="-248.92" y2="91.44" width="0.1524" layer="91"/>
 </segment>
 <segment>
@@
 <label x="-284.48" y="91.44" size="1.4224" layer="95" rot="R90" xref="yes"/>
 </segment>
+<segment>
+<pinref part="R13" gate="G$1" pin="1"/>
+<wire x1="-241.3" y1="104.14" x2="-241.3" y2="106.68" width="0.1524" layer="91"/>
+<label x="-241.3" y="106.68" size="1.4224" layer="95" rot="R90" xref="yes"/>
+</segment>
+<segment>
+<pinref part="IC2" gate="G$1" pin="VCC"/>
+<wire x1="81.28" y1="180.34" x2="88.9" y2="180.34" width="0.1524" layer="91"/>
+<label x="88.9" y="180.34" size="1.4224" layer="95" xref="yes"/>
+</segment>
 </net>
 <net name="N$15" class="0">
@@
 </segment>
 <segment>
-<pinref part="IC2" gate="G$1" pin="RXCA"/>
-<wire x1="81.28" y1="236.22" x2="88.9" y2="236.22" width="0.1524" layer="91"/>
-<label x="88.9" y="236.22" size="1.4224" layer="95" xref="yes"/>
-</segment>
-<segment>
-<pinref part="IC2" gate="G$1" pin="TXCA"/>
-<wire x1="81.28" y1="231.14" x2="88.9" y2="231.14" width="0.1524" layer="91"/>
-<label x="88.9" y="231.14" size="1.4224" layer="95" xref="yes"/>
-</segment>
-<segment>
 <pinref part="JP1" gate="A" pin="9"/>
 <wire x1="-205.74" y1="33.02" x2="-215.9" y2="33.02" width="0.1524" layer="91"/>
 <label x="-215.9" y="33.02" size="1.4224" layer="95" rot="R180" xref="yes"/>
 </segment>
+<segment>
+<pinref part="R21" gate="G$1" pin="1"/>
+<wire x1="-208.28" y1="-12.7" x2="-213.36" y2="-12.7" width="0.1524" layer="91"/>
+<label x="-213.36" y="-12.7" size="1.4224" layer="95" rot="R180" xref="yes"/>
+</segment>
 </net>
 <net name="1228800HZ" class="0">
@@
 <label x="-215.9" y="40.64" size="1.4224" layer="95" rot="R180" xref="yes"/>
 </segment>
+<segment>
+<pinref part="R17" gate="G$1" pin="1"/>
+<wire x1="-208.28" y1="10.16" x2="-213.36" y2="10.16" width="0.1524" layer="91"/>
+<label x="-213.36" y="10.16" size="1.4224" layer="95" rot="R180" xref="yes"/>
+</segment>
 </net>
 <net name="614400HZ" class="0">
@@
 <label x="-215.9" y="38.1" size="1.4224" layer="95" rot="R180" xref="yes"/>
 </segment>
+<segment>
+<pinref part="R18" gate="G$1" pin="1"/>
+<wire x1="-208.28" y1="2.54" x2="-213.36" y2="2.54" width="0.1524" layer="91"/>
+<label x="-213.36" y="2.54" size="1.4224" layer="95" rot="R180" xref="yes"/>
+</segment>
 </net>
 <net name="307200HZ" class="0">
@@
 <label x="-215.9" y="35.56" size="1.4224" layer="95" rot="R180" xref="yes"/>
 </segment>
+<segment>
+<pinref part="R20" gate="G$1" pin="1"/>
+<wire x1="-208.28" y1="-5.08" x2="-213.36" y2="-5.08" width="0.1524" layer="91"/>
+<label x="-213.36" y="-5.08" size="1.4224" layer="95" rot="R180" xref="yes"/>
+</segment>
 </net>
 <net name="2457600HZ" class="0">
@@
 <wire x1="-205.74" y1="43.18" x2="-215.9" y2="43.18" width="0.1524" layer="91"/>
 <label x="-215.9" y="43.18" size="1.4224" layer="95" rot="R180" xref="yes"/>
+</segment>
+<segment>
+<pinref part="R16" gate="G$1" pin="1"/>
+<wire x1="-208.28" y1="17.78" x2="-213.36" y2="17.78" width="0.1524" layer="91"/>
+<label x="-213.36" y="17.78" size="1.4224" layer="95" rot="R180" xref="yes"/>
 </segment>
 </net>
@@
 </segment>
 </net>
+<net name="N$41" class="0">
+<segment>
+<pinref part="IC12" gate="A" pin="CLR"/>
+<pinref part="R13" gate="G$1" pin="2"/>
+<wire x1="-238.76" y1="83.82" x2="-241.3" y2="83.82" width="0.1524" layer="91"/>
+<wire x1="-241.3" y1="83.82" x2="-241.3" y2="93.98" width="0.1524" layer="91"/>
+</segment>
+</net>
+<net name="BAUDRATE_A" class="0">
+<segment>
+<pinref part="R21" gate="G$1" pin="2"/>
+<wire x1="-198.12" y1="-12.7" x2="-195.58" y2="-12.7" width="0.1524" layer="91"/>
+<wire x1="-195.58" y1="-12.7" x2="-195.58" y2="-5.08" width="0.1524" layer="91"/>
+<wire x1="-195.58" y1="-5.08" x2="-195.58" y2="2.54" width="0.1524" layer="91"/>
+<wire x1="-195.58" y1="2.54" x2="-195.58" y2="10.16" width="0.1524" layer="91"/>
+<pinref part="R17" gate="G$1" pin="2"/>
+<wire x1="-198.12" y1="10.16" x2="-195.58" y2="10.16" width="0.1524" layer="91"/>
+<pinref part="R18" gate="G$1" pin="2"/>
+<wire x1="-198.12" y1="2.54" x2="-195.58" y2="2.54" width="0.1524" layer="91"/>
+<junction x="-195.58" y="2.54"/>
+<pinref part="R20" gate="G$1" pin="2"/>
+<wire x1="-198.12" y1="-5.08" x2="-195.58" y2="-5.08" width="0.1524" layer="91"/>
+<junction x="-195.58" y="-5.08"/>
+<wire x1="-195.58" y1="2.54" x2="-190.5" y2="2.54" width="0.1524" layer="91"/>
+<label x="-190.5" y="2.54" size="1.4224" layer="95" xref="yes"/>
+<pinref part="R16" gate="G$1" pin="2"/>
+<wire x1="-198.12" y1="17.78" x2="-195.58" y2="17.78" width="0.1524" layer="91"/>
+<wire x1="-195.58" y1="17.78" x2="-195.58" y2="10.16" width="0.1524" layer="91"/>
+<junction x="-195.58" y="10.16"/>
+</segment>
+<segment>
+<pinref part="IC2" gate="G$1" pin="TXCA"/>
+<wire x1="81.28" y1="231.14" x2="88.9" y2="231.14" width="0.1524" layer="91"/>
+<label x="88.9" y="231.14" size="1.4224" layer="95" xref="yes"/>
+</segment>
+<segment>
+<pinref part="IC2" gate="G$1" pin="RXCA"/>
+<wire x1="81.28" y1="236.22" x2="88.9" y2="236.22" width="0.1524" layer="91"/>
+<label x="88.9" y="236.22" size="1.4224" layer="95" xref="yes"/>
+</segment>
+</net>
