File: hardware/CPU_board/Z80.brd (EAGLE design)
At the start: 167.9 x 122.5 mm, 49 parts, among them IC11 74HCT245DW, IC6 74AC273N, IC9 74HCT138N

Commit message: CPU board and I/O board update
Connections:
- net !IORQ: now also SV2.44
- net M1: now also SV2.43
Routing:
- net M1: track 252.2 -> 299.4 mm, vias 6 -> 8
- net !IORQ: track 209.2 -> 251.9 mm, vias 8 -> 10
- net GND: track 151.5 -> 156.3 mm, vias 14 -> 16
Changed lines of the file:
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@@
 <setting verticaltext="up"/>
 </settings>
-<grid distance="25" unitdist="mil" unit="mil" style="lines" multiple="1" display="no" altdistance="5" altunitdist="mil" altunit="mil"/>
+<grid distance="25" unitdist="mil" unit="mil" style="lines" multiple="1" display="no" altdistance="12.6" altunitdist="mil" altunit="mil"/>
 <layers>
 <layer number="1" name="Top" color="4" fill="1" visible="yes" active="yes"/>
@@
 <contactref element="C4" pad="2"/>
 <contactref element="JP1" pad="1"/>
+<via x="111.6965" y="26.56331875" extent="1-16" drill="0.6" diameter="1.4224" shape="octagon"/>
+<via x="111.6965" y="21.793203125" extent="1-16" drill="0.6" diameter="1.4224" shape="octagon"/>
+<wire x1="111.6965" y1="21.793203125" x2="111.6965" y2="26.56331875" width="0.6096" layer="1"/>
 </signal>
 <signal name="D0">
@@
 <wire x1="53.0225" y1="70.485" x2="53.0225" y2="29.845" width="0.4064" layer="1"/>
 <via x="53.0225" y="29.845" extent="1-16" drill="0.6" diameter="1.4224" shape="octagon"/>
-<wire x1="53.0225" y1="70.485" x2="64.4525" y2="70.485" width="0.4064" layer="16"/>
 <wire x1="51.7525" y1="71.755" x2="53.0225" y2="70.485" width="0.4064" layer="16"/>
 <wire x1="49.53" y1="29.845" x2="53.0225" y2="29.845" width="0.4064" layer="16"/>
+<wire x1="53.0225" y1="70.485" x2="64.4525" y2="70.485" width="0.4064" layer="16"/>
 </signal>
 <signal name="A3">
@@
 <contactref element="IC9" pad="15"/>
 <contactref element="SV2" pad="57"/>
-<wire x1="149.225" y1="19.685" x2="144.4625" y2="19.685" width="0.4064" layer="16"/>
-<wire x1="155.575" y1="24.765" x2="154.305" y2="24.765" width="0.4064" layer="16"/>
-<wire x1="154.305" y1="24.765" x2="149.225" y2="19.685" width="0.4064" layer="16"/>
+<wire x1="146.05" y1="19.685" x2="144.4625" y2="19.685" width="0.4064" layer="16"/>
+<wire x1="155.575" y1="24.765" x2="151.13" y2="24.765" width="0.4064" layer="16"/>
+<wire x1="151.13" y1="24.765" x2="146.05" y2="19.685" width="0.4064" layer="16"/>
 </signal>
 <signal name="CS_2">
@@
 <wire x1="123.825" y1="18.415" x2="123.825" y2="11.43" width="0.4064" layer="16"/>
 <wire x1="122.555" y1="10.16" x2="123.825" y2="11.43" width="0.4064" layer="16"/>
+<contactref element="SV2" pad="44"/>
+<wire x1="136.8425" y1="14.605" x2="141.605" y2="14.605" width="0.4064" layer="16"/>
+<wire x1="141.605" y1="14.605" x2="142.875" y2="15.875" width="0.4064" layer="16"/>
+<wire x1="142.875" y1="15.875" x2="146.05" y2="15.875" width="0.4064" layer="16"/>
+<wire x1="146.05" y1="15.875" x2="153.035" y2="22.86" width="0.4064" layer="16"/>
+<via x="153.035" y="22.86" extent="1-16" drill="0.6" diameter="1.4224" shape="octagon"/>
+<wire x1="153.035" y1="22.86" x2="153.035" y2="39.690040625" width="0.4064" layer="1"/>
+<via x="153.035" y="39.690040625" extent="1-16" drill="0.6" diameter="1.4224" shape="octagon"/>
+<wire x1="158.115" y1="42.545" x2="156.845" y2="41.275" width="0.4064" layer="16"/>
+<wire x1="156.845" y1="41.275" x2="154.619959375" y2="41.275" width="0.4064" layer="16"/>
+<wire x1="154.619959375" y1="41.275" x2="153.035" y2="39.690040625" width="0.4064" layer="16"/>
 </signal>
 <signal name="!MREQ">
@@
 <wire x1="107.315" y1="6.985" x2="107.315" y2="8.255" width="0.4064" layer="16"/>
 <contactref element="IC9" pad="6"/>
-<wire x1="136.8425" y1="9.525" x2="132.715" y2="9.525" width="0.4064" layer="16"/>
-<wire x1="130.175" y1="12.065" x2="132.715" y2="9.525" width="0.4064" layer="16"/>
+<wire x1="136.8425" y1="9.525" x2="134.299959375" y2="9.525" width="0.4064" layer="16"/>
 <wire x1="107.315" y1="8.255" x2="107.315" y2="12.065" width="0.4064" layer="16"/>
 <via x="107.315" y="12.065" extent="1-16" drill="0.6" diameter="1.4224" shape="octagon"/>
-<wire x1="107.315" y1="12.065" x2="130.175" y2="12.065" width="0.4064" layer="1"/>
-<via x="130.175" y="12.065" extent="1-16" drill="0.6" diameter="1.4224" shape="octagon"/>
+<wire x1="107.315" y1="12.065" x2="133.029959375" y2="12.065" width="0.4064" layer="1"/>
+<via x="133.029959375" y="12.065" extent="1-16" drill="0.6" diameter="1.4224" shape="octagon"/>
+<wire x1="133.029959375" y1="12.065" x2="133.029959375" y2="10.795" width="0.4064" layer="16"/>
+<wire x1="133.029959375" y1="10.795" x2="134.299959375" y2="9.525" width="0.4064" layer="16"/>
+<wire x1="133.029959375" y1="12.065" x2="133.029959375" y2="14.284959375" width="0.4064" layer="16"/>
+<wire x1="133.029959375" y1="14.284959375" x2="134.62" y2="15.875" width="0.4064" layer="16"/>
+<wire x1="134.62" y1="15.875" x2="139.065" y2="15.875" width="0.4064" layer="16"/>
+<wire x1="139.065" y1="15.875" x2="141.605" y2="18.415" width="0.4064" layer="16"/>
+<wire x1="141.605" y1="18.415" x2="146.685" y2="18.415" width="0.4064" layer="16"/>
+<wire x1="146.685" y1="18.415" x2="151.13" y2="22.86" width="0.4064" layer="16"/>
+<via x="151.13" y="22.86" extent="1-16" drill="0.6" diameter="1.4224" shape="octagon"/>
+<wire x1="151.13" y1="22.86" x2="151.13" y2="38.1" width="0.4064" layer="1"/>
+<via x="151.13" y="38.1" extent="1-16" drill="0.6" diameter="1.4224" shape="octagon"/>
+<contactref element="SV2" pad="43"/>
+<wire x1="155.575" y1="42.545" x2="153.91891875" y2="42.545" width="0.4064" layer="16"/>
+<wire x1="153.91891875" y1="42.545" x2="151.13" y2="39.75608125" width="0.4064" layer="16"/>
+<wire x1="151.13" y1="38.1" x2="151.13" y2="39.75608125" width="0.4064" layer="16"/>
 </signal>
 <signal name="LOCAL_IO_CS">

Commit message: CPU and I/O board update
Connections:
- removed net 8275_DACK: SV2.2
- removed net RDYIN: SV2.1
- new net IEO: IC2.36, SV2.2
- net INT: now also IC2.37
Routing:
- net IEO: track 0.00 -> 140.8 mm, vias 0 -> 4
- net INT: track 183.6 -> 217.2 mm, vias 2 -> 4
- net GND: track 156.3 -> 173.7 mm, vias 16 -> 18
- net A1: track 202.0 -> 207.2 mm
- net A14: track 225.2 -> 223.3 mm
- net A15: track 253.8 -> 252.3 mm
- net CLK: track 238.6 -> 238.0 mm

Commit message: Bug in CPU board fixed
Connections:
- net GND: now also IC3.11
Changed lines of the file:
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@@
 <via x="99.057459375" y="99.06" extent="1-16" drill="0.6" diameter="1.4224" shape="octagon"/>
 <wire x1="99.057459375" y1="99.06" x2="99.057459375" y2="118.745" width="0.6096" layer="1"/>
+<contactref element="IC3" pad="11"/>
 </signal>
 <signal name="D0">
